File: ZX81Keyboard.sch (KiCad schematic (older format))
At the start: 51 parts, among them J2 Conn_01x05, J3 Conn_01x03, J4 Conn_01x08, SW1 1, SW10 0, SW11 Q, SW12 W, SW13 E, SW14 R, SW15 T, SW16 Y, SW17 U, SW18 I, SW19 O, SW2 2, SW20 P, SW21 A, SW22 S, SW23 D, SW24 F, SW25 G, SW26 H, SW27 J, SW28 K, SW29 L, SW3 3, SW30 NEW_LINE, SW31 SHIFT, SW32 Z, SW33 X, SW34 C, SW35 V, SW36 B, SW37 N, SW38 M, SW39 ., SW4 4, SW40 SPACE, SW5 5, SW6 6, SW7 7, SW8 8, SW9 9

Commit message: Nearing completion.
Changed lines of the file:
@@
 Wire Wire Line
 	5950 5175 5950 5050
-Text Label 8550 1150 3    50   ~ 0
-KD0
-Text Label 8450 1150 3    50   ~ 0
-KD1
-Text Label 8350 1150 3    50   ~ 0
-KD2
-Text Label 8250 1150 3    50   ~ 0
-KD3
-Text Label 8150 1150 3    50   ~ 0
-KD4
-Text Label 8750 1150 3    50   ~ 0
-KA11
-Text Label 8850 1150 3    50   ~ 0
-KA10
-Text Label 8950 1150 3    50   ~ 0
-KA12
-Text Label 9050 1150 3    50   ~ 0
-KA9
-Text Label 9150 1150 3    50   ~ 0
-KA13
-Text Label 9250 1150 3    50   ~ 0
-KA8
-Text Label 9350 1150 3    50   ~ 0
-KA14
-Text Label 9450 1150 3    50   ~ 0
-KA15
 $Comp
 L Connector_Generic:Conn_01x03 J3
@@
 Wire Wire Line
 	7450 5175 7450 5400
+Text GLabel 8150 1150 3    39   Input ~ 0
+KD4
+Text GLabel 8250 1150 3    39   Input ~ 0
+KD3
+Text GLabel 8350 1150 3    39   Input ~ 0
+KD2
+Text GLabel 8450 1150 3    39   Input ~ 0
+KD1
+Text GLabel 8550 1150 3    39   Input ~ 0
+KD0
+Text GLabel 8750 1150 3    39   Input ~ 0
+KA11
+Text GLabel 8850 1150 3    39   Input ~ 0
+KA10
+Text GLabel 8950 1150 3    39   Input ~ 0
+KA12
+Text GLabel 9050 1150 3    39   Input ~ 0
+KA9
+Text GLabel 9150 1150 3    39   Input ~ 0
+KA13
+Text GLabel 9250 1150 3    39   Input ~ 0
+KA8
+Text GLabel 9350 1150 3    39   Input ~ 0
+KA14
+Text GLabel 9450 1150 3    39   Input ~ 0
+KA15
 $EndSCHEMATC
